File: Arduino_OpenTherm_shield.kicad_pcb (KiCad board)
At the start: 2 copper layers, 68.6 x 53.3 mm, 54 parts, among them J1 BOILER, J2 THERM, Q1 MMBT2907A, Q2 MMBT2907A, Q3 MMBT2907A, Q4 MMBT2907A, Q5 MMBT2222A, Q6 MMBT2222A, U1 TPS61040DBV, U2 LTV-817S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

Commit message: Corrected value of the resistance responsible for the High state of the OT bus
Parts:
- R10: value 0R -> 20
- R11: value 47 -> 20
Changed lines of the file:
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@@
 			)
 		)
-		(property "Value" "0R"
+		(property "Value" "20"
 			(at 0 1.43 0)
 			(layer "F.Fab")
@@
 			)
 		)
-		(property "LCSC" "C21189"
+		(property "LCSC" "C22950"
 			(at 0 0 180)
 			(unlocked yes)
@@
 			)
 		)
-		(property "Value" "47"
+		(property "Value" "20"
 			(at 0 1.43 0)
 			(layer "F.Fab")
@@
 			)
 		)
-		(property "LCSC" "C23182"
-			(at 0 0 180)
-			(unlocked yes)
+		(property "LCSC" "C22950"
+			(at 0 0 180)
+			(unlocked yes)

Commit message: updated bom list
Parts:
- U1: value TPS61040DBV -> MT3540-F23
Changed lines of the file:
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@@
 			)
 		)
-		(property "Value" "TPS61040DBV"
+		(property "Value" "MT3540-F23"
 			(at 0 2.4 0)
 			(layer "F.Fab")
@@
 			)
 		)
-		(property "LCSC" "C7722"
+		(property "LCSC" "C181783"
 			(at 0 0 0)
 			(unlocked yes)

Commit message: HW rev 1.2 [fixed translation of MASTER_IN signal logic levels]
Parts:
- added D9: 8V2, footprints:D_SOD-123, F.Cu at (85.1, 62.4)
- R12: value 20k -> 10k
- R13: value 10k -> 150k
- R17: value 1k1 -> 1k8
- moved R12 4.89 mm to (85.1, 66.4)
- moved R13 4.09 mm to (85.9, 68.8), turned to 0 degrees
- moved R9 1.32 mm to (87.6, 67.2), turned to 0 degrees
- renumbered D9 to D10, D10 to D11, D11 to D12
Connections:
- J2 pad 1: Net-(J2-Pin_1) -> Net-(D9-K)
- Q3 pad 3: Net-(J2-Pin_1) -> Net-(D9-K)
- R12 pad 2: Net-(J2-Pin_1) -> Net-(D9-A)
- TP4 pad 1: Net-(J2-Pin_1) -> Net-(D9-K)
Routing:
- net Net-(J2-Pin_1): track 16.1 -> 0.00 mm
- net Net-(D9-K): track 0.00 -> 16.1 mm
- net Net-(Q6-B): track 15.6 -> 17.8 mm
- net GND: track 17.4 -> 15.8 mm
- net Net-(D9-A): track 0.00 -> 1.59 mm

Commit message: RxB LED brightness adjusted
Parts:
- R17: value 1k8 -> 5k1
Changed lines of the file:
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@@
 			)
 		)
-		(property "Value" "1k8"
+		(property "Value" "5k1"
 			(at 0 1.43 90)
 			(layer "F.Fab")
@@
 			)
 		)
-		(property "LCSC" "C4177"
+		(property "LCSC" "C23186"
 			(at 0 0 90)
 			(unlocked yes)
